File: PCB/ZBoard V1.kicad_pcb (KiCad board)
At the start: 2 copper layers, 333 x 119 mm, 180 parts, among them SW1 SW_Push, SW10 SW_Push, SW11 SW_Push, SW12 SW_Push, SW13 SW_Push, SW14 SW_Push, SW15 SW_Push, SW16 SW_Push, SW17 SW_Push, SW18 SW_Push, SW19 SW_Push, SW2 SW_Push, SW20 SW_Push, SW21 SW_Push, SW22 SW_Push, SW23 SW_Push, SW24 SW_Push, SW25 SW_Push, SW26 SW_Push, SW27 SW_Push, SW28 SW_Push, SW29 SW_Push, SW3 SW_Push, SW30 SW_Push, SW31 SW_Push, SW32 SW_Push, SW33 SW_Push, SW34 SW_Push, SW35 SW_Push, SW36 SW_Push, SW37 SW_Push, SW38 SW_Push, SW39 SW_Push, SW4 SW_Push, SW40 SW_Push, SW41 SW_Push, SW42 SW_Push, SW43 SW_Push, SW44 SW_Push, SW45 SW_Push, SW46 SW_Push, SW47 SW_Push, SW48 SW_Push, SW49 SW_Push, SW5 SW_Push, SW50 SW_Push, SW51 SW_Push, SW52 SW_Push, SW53 SW_Push, SW54 SW_Push, SW55 SW_Push, SW56 SW_Push, SW57 SW_Push, SW58 SW_Push, SW59 SW_Push, SW6 SW_Push, SW60 SW_Push, SW61 SW_Push, SW62 SW_Push, SW63 SW_Push, SW64 SW_Push, SW65 SW_Push, SW66 SW_Push, SW67 SW_Push, SW68 SW_Push, SW69 SW_Push, SW7 SW_Push, SW70 SW_Push, SW71 SW_Push, SW72 SW_Push, SW73 SW_Push, SW74 SW_Push, SW75 SW_Push, SW76 SW_Push, SW77 SW_Push, SW78 SW_Push, SW79 SW_Push, SW8 SW_Push, SW80 SW_Push, SW81 SW_Push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

Commit message: Fixed pinouts, fixed firmware
Connections:
- net GNDBAT renamed BATGND
- U1 pad 6: /ROW1 -> /SCL
- U1 pad 9: /SCK -> /ROW1
- U2 pad 12: /SCK -> /SCL
Routing:
- net /SCL: track 0.00 -> 50.4 mm, vias 0 -> 1
- net /SCK: track 46.4 -> 0.00 mm, vias 1 -> 0
- net /ROW1: track 312.9 -> 325.7 mm
- net +5V: track 48.3 -> 59.5 mm, vias 2 -> 3
- net /COL1: track 493.9 -> 494.5 mm

Commit message: Beginning transition to wired using Orpheus Pico
Parts:
- removed R1: 806k, MFR-25FRF52-806k:MFR-25FRF52-806k
- removed R2: 2M, MFR-25FRF52-2M:MFR-25FRF52-2M
- removed TP1: BAT, TestPoint:TestPoint_Pad_D2.0mm
- removed TP2: GND, TestPoint:TestPoint_Pad_2.0x2.0mm
- removed U1: XIAO-nRF52840-SMD, Modified-XIAO:modified-XIAO-nRF52840-SMD
- removed U2: MCP23017-E_SP, MCP23017_GPIO:MCP23107_GPIO
- added G***: LOGO, Silkscreen:ZHub-V1-Logo, F.Cu at (137.5, 76.7)
- added U3: Pico, MCU_RaspberryPi_and_Boards:RPi_Pico_SMD_TH, F.Cu at (332.8, 38.1)
Routing:
- net BATGND: track 78.1 -> 0.00 mm, vias 1 -> 0
- net GND: track 77.0 -> 2.67 mm, vias 0 -> 2
- net /VBAT: track 69.9 -> 0.00 mm, vias 1 -> 0
- net +5V: track 59.5 -> 0.00 mm, vias 3 -> 0
- net /COL11: track 203.4 -> 261.1 mm, vias 1 -> 2
- net /COL9: track 345.6 -> 289.7 mm, vias 1 -> 2
- net /ROW6: track 434.2 -> 381.8 mm, vias 11 -> 10
- net /SCL: track 50.4 -> 0.00 mm, vias 1 -> 0
- net /BT_PIN: track 47.7 -> 0.00 mm, vias 1 -> 0
- net /COL8: track 365.9 -> 319.2 mm, vias 1 -> 2
- net /SDA: track 44.4 -> 0.00 mm, vias 1 -> 0
- net /COL1: track 494.5 -> 528.0 mm, vias 5 -> 1
- net /COL16: track 24.6 -> 53.2 mm
- net /COL12: track 190.0 -> 211.9 mm, vias 1 -> 2
- net /COL13: track 167.0 -> 188.6 mm, vias 1 -> 2
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- added copper zone on B.Cu, net GND
